Commit message: Added new description, usb camera, in aramis

File: robots/aramis_description.xacro (robot description, xacro)
@@ -4,4 +4,5 @@
     <xacro:include filename="$(find aramis_description)/robots/suporte_aramis_description.URDF"/>
     <xacro:include filename="$(find aramis_description)/robots/sensor_sonar_pioneer.urdf.xacro"/>
+    <xacro:include filename="$(find aramis_description)/robots/sensor_camera_usb_pioneer.urdf.xacro"/>
     <xacro:include filename="$(find pr2_description)/urdf/sensors/kinect_camera.urdf.xacro" />
     <xacro:include filename="$(find pr2_description)/urdf/common.xacro" />
@@ -26,4 +27,8 @@
                     <origin rpy="0 1.57 1.57"  xyz="0.170 0.087 0.0"/>
     </kinect_camera_v0>
+    <camera_usb name="camera_usb" parent="suporte_kinect">
+                    <!-- <origin rpy="0 -3.9246 1.57"  xyz="0.170 0.067 -0.035"/> -->
+                    <origin rpy="1.57 0 3.14"  xyz="0.275 0.0 0.060"/>
+    </camera_usb>
     <sonar_pioneer name="sonar_0" parent="base_link">
         <origin xyz="0.069 0.130 0.209" rpy="0 0 1.5708"/>
